Commit message: Modified the original driver for lab setup and applications
realsense2_description/launch/view_model.launch.py: Added a topic remapping for the robot state publisher to avoid conflicts with the KUKA URDF and commented out the RViz2 Node from the launch

realsense2_description/urdf/test_d435_camera.urdf.xacro: Modified the default location of the URDF to match the location of the Realsense D435 in the lab and changed the parent link to root

realsense2_camera/launch/combined_launch.py: Created a launch file to launch the Driver and URDF/Transform publisher simultaneously

File: realsense2_description/urdf/test_d435_camera.urdf.xacro (robot description, xacro)
@@ -5,7 +5,8 @@
   <xacro:arg name="use_mesh" default="true" />
   <xacro:include filename="$(find realsense2_description)/urdf/_d435.urdf.xacro" />
-  <link name="base_link" />
-  <xacro:sensor_d435 parent="base_link" use_nominal_extrinsics="$(arg use_nominal_extrinsics)" add_plug="$(arg add_plug)" use_mesh="$(arg use_mesh)">
-    <origin xyz="0 0 0" rpy="0 0 0"/>
+  <!-- Changed the spawning location of the Realsense Camera URDF and changed the parent link to "root" -->
+  <link name="root" />
+  <xacro:sensor_d435 name="camera" parent="root" use_nominal_extrinsics="$(arg use_nominal_extrinsics)" add_plug="$(arg add_plug)" use_mesh="$(arg use_mesh)">
+    <origin xyz="-0.84 0.44 1.19" rpy="0.0 0.0 0.0"/>
   </xacro:sensor_d435>
 </robot>
